Commit message: updated xarco for pioneer3dx for jade where error occurs on default_interia macro not existing

File: rocs_simulation/urdf_model/defs/pioneer3dx_new.xacro (robot description, xacro)
@@ -1,4 +1,5 @@
 <?xml version='1.0' encoding='UTF-8'?>
 <robot xmlns:sensor="http://playerstage.sourceforge.net/gazebo/xmlschema/#sensor" xmlns:controller="http://playerstage.sourceforge.net/gazebo/xmlschema/#controller" xmlns:interface="http://playerstage.sourceforge.net/gazebo/xmlschema/#interface" xmlns:xacro="http://ros.org/wiki/xacro" name="pioneer3dx">
+  <xacro:macro name="default_inertial">
   <xacro:include filename="$(find rocs_simulation)/urdf_model/defs/pioneer3dx_wheel.xacro"/>
 <!-- Chassis -->
@@ -231,5 +232,4 @@
 <xacro:macro name="easy_cylinder" params="name radius length *vorigin *corigin *material">
 	<link name="${name}">
-		<xacro:default_inertia/>
 	<visual>
 		<xacro:insert_block name="vorigin"/>
@@ -249,5 +249,4 @@
 <xacro:macro name="easy_box" params="name size *vorigin *corigin *material">
 	<link name="${name}">
-		<xacro:default_inertia/>
 		<visual>
 			<xacro:insert_block name="vorigin"/>

Commit message: fixed model and setupbash file for multiple distros and navigation

File: rocs_simulation/urdf_model/defs/pioneer3dx_new.xacro (robot description, xacro)
@@ -1,5 +1,4 @@
 <?xml version='1.0' encoding='UTF-8'?>
 <robot xmlns:sensor="http://playerstage.sourceforge.net/gazebo/xmlschema/#sensor" xmlns:controller="http://playerstage.sourceforge.net/gazebo/xmlschema/#controller" xmlns:interface="http://playerstage.sourceforge.net/gazebo/xmlschema/#interface" xmlns:xacro="http://ros.org/wiki/xacro" name="pioneer3dx">
-  <xacro:macro name="default_inertial">
   <xacro:include filename="$(find rocs_simulation)/urdf_model/defs/pioneer3dx_wheel.xacro"/>
 <!-- Chassis -->
